File: Battery_Charger.sch (KiCad schematic (older format))
At the start: 13 parts, among them J1 CONN_01X15, U1 TCA9548A_TSSOP, U2 LTC2943, U3 LTC2943

Commit message: Add files via upload
Parts:
- removed J1: CONN_01X15, symbol CONN_01X15
- removed K?: G6E, Relays_THT:Relay_SPDT_OMRON-G6E, symbol G6E
- removed U1: TCA9548A_TSSOP, Housings_SSOP:TSSOP-24_4.4x7.8mm_Pitch0.65mm, symbol TCA9548A_TSSOP
- removed U2, U3: LTC2943, symbol LTC2943
- removed U?: LM317_SOT223, symbol LM317_SOT223
- added C1, C5: 1uF, Capacitors_SMD:C_0603_HandSoldering, symbol C
- added C3, C4: C, Capacitors_SMD:C_0603_HandSoldering, symbol C
- added D1, D2: D, Diodes_SMD:D_0603, symbol D
- added J1: Screw_Terminal_1x02, Connectors_Terminal_Blocks:TerminalBlock_Pheonix_MKDS1.5-2pol, symbol Screw_Terminal_1x02
- added J2: CONN_01X14, Connectors_Molex:Molex_KK-6410-14_14x2.54mm_Straight, symbol CONN_01X14
- added K1, K2: G6E, Relays_THT:Relay_SPDT_OMRON-G6E, symbol G6E
- added Q1, Q2: Q_NPN_BCE, TO_SOT_Packages_SMD:SOT-23, symbol Q_NPN_BCE
- added R10: 1, Resistors_SMD:R_1812_HandSoldering, symbol R
- added R11, R9: 0.05, Resistors_SMD:R_2512_HandSoldering, symbol R
- added R12, R13: R, Resistors_SMD:R_1812_HandSoldering, symbol R
- added R8: 1k, Resistors_SMD:R_0603_HandSoldering, symbol R
- added U1, U4: LTC2943, Housings_DFN_QFN:DFN-8-1EP_3x3mm_Pitch0.5mm, symbol LTC2943-RESCUE-Battery_Charger
- added U2: TCA9548A_QFN, Housings_SSOP:TSSOP-24_4.4x7.8mm_Pitch0.65mm, symbol TCA9548A_QFN
- added U3, U5: LM317AT, TO_SOT_Packages_THT:TO-220_Horizontal, symbol LM317AT
- R1: value R -> 2k; footprint (none) -> Resistors_SMD:R_0603_HandSoldering
- R2, R3, R5: value R -> 10k; footprint (none) -> Resistors_SMD:R_0603_HandSoldering
- R4: value 2k -> 10k; footprint (none) -> Resistors_SMD:R_0603_HandSoldering
- R6: value R -> 1; footprint (none) -> Resistors_SMD:R_1812_HandSoldering
- R7: value R -> 1k; footprint (none) -> Resistors_SMD:R_0603_HandSoldering
Connections:
- net labels added: +5V, 5V, SCL_M, SCO, SDA_M, Vbat_1, Vbat_2, rel_1, rel_2, ~ALCC, ~RST
- net labels removed: +3.3V, M_SCL, M_SDA, SC0, SD0, Vbat_+, Vcc, Vcc_3.3, ~ALCC_2, ~M_RST
- wire segments 48 -> 114
- no-connect marks 12 -> 13
